Commit message: change model

File: catkin_ws/src/me212bot/model/me212bot.xacro (robot description, xacro)
@@ -1,5 +1,5 @@
 <?xml version="1.0"?>
 <robot xmlns:xacro="http://www.ros.org/wiki/xacro" name="me212bot">
-<link name="robot_base">
+<link name="base_link">
     <visual>
         <geometry>
